File: serializer.kicad_sch (KiCad schematic)
At the start: 33 parts, among them U6 MAX96717GTJ_VY+, Y1 Resonator_25MHz_ABM8G

Commit message: [#66847] Update config resistors
Parts:
- R21: value R_80k6_0402 -> R_10k_0402; symbol antmicroResistors0402:R_80k6_0402 -> antmicroResistors0402:R_10k_0402; MPN CR0402-FX-8062GLF -> CR0402-FX-1002GLF; Val 80k6 -> 10k; now fitted; now in the parts list
- R22: now not fitted; now left out of the parts list
Other:
- note added: "CFG0 - I2C address config R1 = OPEN, R2 = 10k I2C; Address = 0x40 (7-bit); Clock= RoR"
- note added: "CFG1 - GMSL mode config R1 = 10k, R2 = OPEN mode = COAX 6Gbps; Pixel mode"
- note removed: "CFG0 - I2C address config R1 = OPEN, R2 = 10k address = 0x80"
- note removed: "CFG1 - GMSL mode config R1 = OPEN, R2 = 10k mode = COAX GMSL2 6Gbps"
Changed lines of the file:
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@@
     )
   )
-  (text "CFG0 - I2C address config\nR1 = OPEN, R2 = 10k\naddress = 0x80"
-    (at 36.83 187.325 0)
+  (text "CFG0 - I2C address config\nR1 = OPEN, R2 = 10k\nI2C; Address = 0x40 (7-bit); \nClock= RoR"
+    (at 38.1 187.325 0)
     (effects (font (size 1.27 1.27)) (justify left bottom))
   )
@@
     (effects (font (size 1.27 1.27)) (justify left bottom))
   )
-  (text "CFG1 - GMSL mode config\nR1 = OPEN, R2 = 10k\nmode = COAX GMSL2 6Gbps"
+  (text "CFG1 - GMSL mode config\nR1 = 10k, R2 = OPEN\nmode = COAX 6Gbps; Pixel mode"
     (at 72.39 187.325 0)
     (effects (font (size 1.27 1.27)) (justify left bottom))
@@
     )
   )
-  (symbol (lib_id "antmicroResistors0402:R_80k6_0402") (at 82.55 201.93 90) (unit 1)
-    (in_bom no) (on_board yes) (dnp yes)
-    (property "Reference" "R21" (at 84.455 198.12 90)
-      (effects (font (size 1.27 1.27) (thickness 0.15)) (justify right))
-    )
-    (property "Value" "R_80k6_0402" (at 95.25 181.61 0)
+  (symbol (lib_id "antmicroResistors0402:R_10k_0402") (at 82.55 201.93 90) (unit 1)
+    (in_bom yes) (on_board yes) (dnp no) (fields_autoplaced)
+    (property "Reference" "R21" (at 85.09 198.12 90)
+      (effects (font (size 1.27 1.27) (thickness 0.15)) (justify right))
+    )
+    (property "Value" "R_10k_0402" (at 95.25 181.61 0)
       (effects (font (size 1.27 1.27) (thickness 0.15)) (justify left bottom) hide)
     )
@@
       (effects (font (size 1.27 1.27) (thickness 0.15)) (justify left bottom) hide)
     )
-    (property "MPN" "CR0402-FX-8062GLF" (at 102.87 181.61 0)
+    (property "MPN" "CR0402-FX-1002GLF" (at 102.87 181.61 0)
       (effects (font (size 1.27 1.27) (thickness 0.15)) (justify left bottom) hide)
     )
@@
       (effects (font (size 1.27 1.27) (thickness 0.15)) (justify left bottom) hide)
     )
-    (property "Val" "80k6" (at 84.455 200.66 90)
+    (property "Val" "10k" (at 85.09 200.66 90)
       (effects (font (size 1.27 1.27) (thickness 0.15)) (justify right))
     )
@@
   )
   (symbol (lib_id "antmicroResistors0402:R_10k_0402") (at 82.55 212.09 90) (unit 1)
-    (in_bom yes) (on_board yes) (dnp no)
+    (in_bom no) (on_board yes) (dnp yes)
     (property "Reference" "R22" (at 84.455 208.28 90)
       (effects (font (size 1.27 1.27) (thickness 0.15)) (justify right))
